File: LoRa Environmental Sensors/LoRa Environmental Sensors.sch (KiCad schematic (older format))
At the start: 8 parts, among them U1 BME280, U2 ATtiny85-20SU, U3 RFM95W-868S2

Commit message: update hardware
Parts:
- removed R1: 4.7k, Resistor_SMD:R_0603_1608Metric_Pad1.05x0.95mm_HandSolder, symbol Device:R
- added J1: SPI, Connector_PinHeader_2.54mm:PinHeader_2x03_P2.54mm_Vertical, symbol Connector_Generic:Conn_02x03_Odd_Even
- added R2: 4.7k, Resistor_SMD:R_0603_1608Metric_Pad1.05x0.95mm_HandSolder, symbol Device:R
- C1, C2: value C -> 0.1uF
- renumbered R2 to R1
Connections:
- net labels added: AtTiny_Reset, VCC
- net labels removed: +3V3
- wire segments 7 -> 20
- no-connect marks 9 -> 8
Other:
- note added: "Power"
- note added: "SPI Interface"
- note added: "VCC Decoupling Capacitors"
- moved on the sheet: U2

Commit message: update env sensor
Changed lines of the file:
@@
 MOSI
 Text Label 3150 4000 0    50   ~ 0
-MOSI
+MISO
 NoConn ~ 8800 4600
 $Comp
