File: atmega328-sensor/sensor_atmega328.sch (KiCad schematic (older format))
At the start: 13 parts, among them J1 Input, J2 Gnd, J3 Output, J4 Conn_01x04, U1 L7805, U2 ATmega328P-PU, U3 RFM95W-868S2, Y1 Crystal

Commit message: update env sensor
Parts:
- removed AE1: Antenna, symbol Device:Antenna
- added C5, C6, C7, C8, C9: 100n, Capacitor_THT:C_Disc_D3.0mm_W1.6mm_P2.50mm, symbol Device:C
- added J5: Conn_01x07, Connector_PinHeader_2.54mm:PinHeader_1x07_P2.54mm_Vertical, symbol Connector_Generic:Conn_01x07
- added J6: Conn_01x06, Connector_PinHeader_2.54mm:PinHeader_1x06_P2.54mm_Vertical, symbol Connector_Generic:Conn_01x06
- added R1: 10k, Resistor_THT:R_Axial_DIN0309_L9.0mm_D3.2mm_P12.70mm_Horizontal, symbol Device:R
- C3, C4: footprint Capacitor_THT:C_Disc_D6<<.0mm_W2.5mm_P5.00mm -> Capacitor_THT:C_Disc_D5.0mm_W2.5mm_P5.00mm
- J4: footprint (none) -> Connector_PinHeader_2.54mm:PinHeader_1x04_P2.54mm_Vertical
- U3: footprint (none) -> RF_Module:HOPERF_RFM9XW_THT
Connections:
- net labels added: +3V3, Reset, RxD, SCL, SDA, TxD
- wire segments 18 -> 31
- no-connect marks 19 -> 20
Other:
- note added: "16Mhz Clock"
- note added: "3.3V Regulator"
- note added: "BME 280"
- note added: "CO2-Sensor"
- note added: "FTDI"
- note added: "Hope RFM952 Lora Module"
- note added: "VCC Decoupling Capacitors"
- moved on the sheet: U2
